Commit message: Chỉnh lỗi robot trôi trong gazebo, thêm camera

File: diff_robot/urdf/diff_robot.urdf (robot description, URDF)
Before this commit: robot diff_robot, 5 links, 4 joints
Links:
- added link esp32_cam_link, mass 0.01; collision mesh filename=package://diff_robot/meshes/esp32_cam_link.STL; visual mesh filename=package://diff_robot/meshes/esp32_cam_link.STL
- link base_footprint: mass 0.142039932145577 -> 0.178
- link base_link: mass 0.440554283125895 -> 0.677
- link caster_wheel: mass 0.122994969459015 -> 0.122
- link left_wheel: mass 0.0790315658072254 -> 0.039
- link right_wheel: mass 0.0790315658065018 -> 0.039
Joints:
- added joint esp32_cam_joint: type fixed, parent base_link, child esp32_cam_link, origin xyz=0.20857 0.0083034 -0.043987 rpy=-3.1416 0 0, axis 0 0 0
- joint base_link_joint: origin xyz=0.000218079198520476 0 0.0325488105635752 rpy=0 0 0 -> xyz=0 0 0.03255 rpy=3.1416 0 0
- joint caster_wheel_joint: axis 0 0 0 -> 0 0 1; origin xyz=0.165 0 -0.0173 rpy=0 0 0 -> xyz=0.165 0 0.0208 rpy=-3.1416 0 0
- joint left_wheel_joint: origin xyz=0 0.1015 0 rpy=1.5708 0 3.1416 -> xyz=0 -0.1168 0 rpy=-1.5708 0 -3.1416
- joint right_wheel_joint: origin xyz=-0.0001512 -0.1015 0.00082881 rpy=1.5708 0 3.1416 -> xyz=0 0.1168 0 rpy=-1.5708 0 -3.1416

Commit message: feat(urdf): update robot's URDF with IMU

File: diff_robot/urdf/diff_robot.urdf (robot description, URDF)
Before this commit: robot diff_robot, 6 links, 5 joints
Links:
- added link imu_link, mass 0.00071663; collision mesh filename=package://diff_robot/meshes/imu_link.STL; visual mesh filename=package://diff_robot/meshes/imu_link.STL
- link base_link: mass 0.677 -> 0.667
- link esp32_cam_link: mass 0.01 -> 0.0098347
Joints:
- added joint imu_link_joint: type fixed, parent base_link, child imu_link, origin xyz=0.035146 -0.069394 0.035 rpy=0 0 0, axis 0 0 0
- joint base_link_joint: origin xyz=0 0 0.03255 rpy=3.1416 0 0 -> xyz=0 0 0.03255 rpy=0 0 0
- joint caster_wheel_joint: axis 0 0 1 -> 0 0 0; origin xyz=0.165 0 0.0208 rpy=-3.1416 0 0 -> xyz=0.165 0 -0.0208 rpy=0 0 0
- joint esp32_cam_joint: origin xyz=0.20857 0.0083034 -0.043987 rpy=-3.1416 0 0 -> xyz=0.20857 -0.0083034 0.043987 rpy=0 0 0
- joint left_wheel_joint: origin xyz=0 -0.1168 0 rpy=-1.5708 0 -3.1416 -> xyz=0 0.1168 0 rpy=1.5708 0 3.1416
- joint right_wheel_joint: origin xyz=0 0.1168 0 rpy=-1.5708 0 -3.1416 -> xyz=0 -0.1168 0 rpy=1.5708 0 3.1416
